File: Electronics/Patrol Bot Circuitry/Patrol Bot Circuitry.kicad_pcb (KiCad board)
At the start: 2 copper layers, 101 x 89.5 mm, 40 parts, among them J1 Left_Motor, J2 Right_Motor, J3 Battery, J4 AC_DC_10V, J5 Servo Motor, Q1 IRF4905, Q2 IRF4905, Q3 IRF4905, Q4 IRLZ44N, U1 ROB-14450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

Commit message: CAD Upload 1
Parts:
- moved J1 2.50 mm to (118.0, 72.0)
- moved J2 2.50 mm to (106.5, 72.0)
Routing:
- net Net-(J1-Pad2): track 10.9 -> 12.4 mm
- net Net-(J1-Pad1): track 12.0 -> 13.1 mm
- net Net-(J2-Pad2): track 10.5 -> 9.48 mm
- net Net-(J2-Pad1): track 9.46 -> 10.3 mm
- net (no net): vias 0 -> 4
Changed lines of the file:
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@@
     (thickness 1.6)
     (drawings 4)
-    (tracks 288)
+    (tracks 294)
     (zones 0)
     (modules 40)
@@
   (page A4)
   (layers
-    (0 F.Cu signal)
-    (31 B.Cu signal)
+    (0 F.Cu signal hide)
+    (31 B.Cu signal hide)
     (32 B.Adhes user)
     (33 F.Adhes user)
@@
   )
   (setup
-    (last_trace_width 2.2)
+    (last_trace_width 0.25)
     (user_trace_width 1)
     (user_trace_width 2.2)
@@
   )
   (module TerminalBlock_Phoenix:TerminalBlock_Phoenix_MKDS-1,5-2-5.08_1x02_P5.08mm_Horizontal (layer F.Cu)
-    (at 104 72 180)
+    (at 106.5 72 180)
     (descr "Terminal Block Phoenix MKDS-1,5-2-5.08, 2 pins, pitch 5.08mm, size 10.2x9.8mm^2, drill diamater 1.3mm, pad diameter 2.6mm, see http://www.farnell.com/datasheets/100425.pdf, script-generated using https://github.com/pointhi/kicad-footprint-generator/scripts/TerminalBlock_Phoenix")
     (tags "THT Terminal Block Phoenix MKDS-1,5-2-5.08 pitch 5.08mm size 10.2x9.8mm^2 drill 1.3mm pad 2.6mm")
@@
   )
   (module TerminalBlock_Phoenix:TerminalBlock_Phoenix_MKDS-1,5-2-5.08_1x02_P5.08mm_Horizontal (layer F.Cu)
-    (at 115.5 72 180)
+    (at 118 72 180)
     (descr "Terminal Block Phoenix MKDS-1,5-2-5.08, 2 pins, pitch 5.08mm, size 10.2x9.8mm^2, drill diamater 1.3mm, pad diameter 2.6mm, see http://www.farnell.com/datasheets/100425.pdf, script-generated using https://github.com/pointhi/kicad-footprint-generator/scripts/TerminalBlock_Phoenix")
     (tags "THT Terminal Block Phoenix MKDS-1,5-2-5.08 pitch 5.08mm size 10.2x9.8mm^2 drill 1.3mm pad 2.6mm")
@@
   (gr_line (start 91.5 153.5) (end 192.5 153.5) (layer Edge.Cuts) (width 0.1))
   (gr_line (start 91.5 64) (end 91.5 153.5) (layer Edge.Cuts) (width 0.1))
+  (via (at 189 67.5) (size 4.5) (drill 4) (layers F.Cu B.Cu) (net 0))
+  (via (at 95 67.5) (size 4.5) (drill 4) (layers F.Cu B.Cu) (net 0))
+  (via (at 95 150) (size 4.5) (drill 4) (layers F.Cu B.Cu) (net 0))
+  (via (at 189 150) (size 4.5) (drill 4) (layers F.Cu B.Cu) (net 0))
   (via (at 167 91) (size 2) (drill 1.5) (layers F.Cu B.Cu) (net 1))
   (via (at 170.5 91) (size 2) (drill 1.5) (layers F.Cu B.Cu) (net 1))
@@
   (segment (start 108.14 147.4) (end 110.54 145) (width 0.25) (layer F.Cu) (net 8))
   (segment (start 106 147.4) (end 108.14 147.4) (width 0.25) (layer F.Cu) (net 8))
-  (segment (start 106.73 75.69) (end 110.42 72) (width 2.2) (layer F.Cu) (net 9))
-  (segment (start 106.73 81.38) (end 106.73 75.69) (width 2.2) (layer F.Cu) (net 9))
-  (segment (start 109.27 78.23) (end 115.5 72) (width 2.2) (layer F.Cu) (net 10))
-  (segment (start 109.27 81.38) (end 109.27 78.23) (width 2.2) (layer F.Cu) (net 10))
-  (segment (start 101.65 74.73) (end 98.92 72) (width 2.2) (layer F.Cu) (net 11))
-  (segment (start 101.65 81.38) (end 101.65 74.73) (width 2.2) (layer F.Cu) (net 11))
-  (segment (start 104.19 72.19) (end 104 72) (width 2.2) (layer F.Cu) (net 12))
-  (segment (start 104.19 81.38) (end 104.19 72.19) (width 2.2) (layer F.Cu) (net 12))
+  (segment (start 112.105874 72) (end 112.92 72) (width 2.2) (layer F.Cu) (net 9))
+  (segment (start 106.73 77.375874) (end 112.105874 72) (width 2.2) (layer F.Cu) (net 9))
+  (segment (start 106.73 81.38) (end 106.73 77.375874) (width 2.2) (layer F.Cu) (net 9))
+  (segment (start 117.800798 72) (end 118 72) (width 2.2) (layer F.Cu) (net 10))
+  (segment (start 109.27 80.530798) (end 117.800798 72) (width 2.2) (layer F.Cu) (net 10))
+  (segment (start 109.27 81.38) (end 109.27 80.530798) (width 2.2) (layer F.Cu) (net 10))
+  (segment (start 101.65 72.23) (end 101.42 72) (width 2.2) (layer F.Cu) (net 11))
+  (segment (start 101.65 81.38) (end 101.65 72.23) (width 2.2) (layer F.Cu) (net 11))
+  (segment (start 104.19 74.31) (end 106.5 72) (width 2.2) (layer F.Cu) (net 12))
+  (segment (start 104.19 81.38) (end 104.19 74.31) (width 2.2) (layer F.Cu) (net 12))
   (segment (start 107.92 135.58) (end 108 135.5) (width 2.2) (layer B.Cu) (net 13))
   (segment (start 98.5 135.58) (end 107.92 135.58) (width 2.2) (layer B.Cu) (net 13))
@@
     (polygon
       (pts
-        (xy 192.5 153.5) (xy 91.5 153.5) (xy 91.5 64) (xy 192.5 64)
+        (xy 192.5 153.5) (xy 91.5 153.5) (xy 91.5 65.25) (xy 192.5 64)
       )
     )
