File: Model 1/Electronics/Patrol Bot Circuitry/Patrol Bot Circuitry.sch (KiCad schematic (older format))
At the start: 46 parts, among them J1 Left_Motor, J2 Right_Motor, J3 Battery, J4 AC_DC_10V, J5 Servo Motor, Q1 Q_NMOS_GSD, Q2 Q_PMOS_GSD, Q3 Q_NMOS_GSD, Q4 Q_PMOS_GSD, Q5 Q_PMOS_GSD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

Commit message: Save
Parts:
- R2: value 620K -> 680K
Connections:
- net 5V is gone; now on net +5V: U10.1 (VCC), U2.1 (VDD), U8.1 (VCC), U9.1 (VCC)
Changed lines of the file:
@@
 P 2000 1550
 F 0 "R2" H 2070 1596 50  0000 L CNN
-F 1 "620K" H 2070 1505 50  0000 L CNN
+F 1 "680K" H 2070 1505 50  0000 L CNN
 F 2 "Resistor_SMD:R_0603_1608Metric" V 1930 1550 50  0001 C CNN
 F 3 "~" H 2000 1550 50  0001 C CNN
@@
 $EndComp
 $Comp
-L power:+5V #PWR0109
-U 1 1 61E78D4E
-P 3250 3650
-F 0 "#PWR0109" H 3250 3500 50  0001 C CNN
-F 1 "+5V" H 3265 3823 50  0000 C CNN
-F 2 "" H 3250 3650 50  0001 C CNN
-F 3 "" H 3250 3650 50  0001 C CNN
-	1    3250 3650
-	1    0    0    -1
-$EndComp
-$Comp
 L power:+5V #PWR0108
 U 1 1 61E7857F
@@
 $EndComp
 $Comp
-L power:+5V #PWR?
+L power:+5V #PWR0111
 U 1 1 6207BCFE
 P 1750 5300
-F 0 "#PWR?" H 1750 5150 50  0001 C CNN
+F 0 "#PWR0111" H 1750 5150 50  0001 C CNN
 F 1 "+5V" H 1765 5473 50  0000 C CNN
 F 2 "" H 1750 5300 50  0001 C CNN
@@
 Wire Wire Line
 	1750 5300 2000 5300
+Text Label 5950 2450 0    50   ~ 0
+5V
+Text Label 3250 3650 2    50   ~ 0
+5V
 $EndSCHEMATC
